File: kicad-nerdYcontroller/power-and-usb.kicad_sch (KiCad schematic)
At the start: 12 parts, among them J201 S2B-PH-SM4-TB, P201 USB_C_Plug_USB2.0, U201 AMS1117-3.3

Commit message: fixing missing usb-c 2-way connectivity
Connections:
- net USBC-D+: now also P201.B6 (D+)
- net USBC-D-: now also P201.B7 (D-)
Changed lines of the file:
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@@
+	)
+	(junction
+		(at 74.93 52.07)
+		(diameter 0)
+		(color 0 0 0 0)
 	)
 	(junction
@@
 	)
 	(junction
+		(at 66.04 57.15)
+		(diameter 0)
+		(color 0 0 0 0)
+	)
+	(junction
 		(at 97.79 48.26)
 		(diameter 0)
@@
 	(wire
 		(pts
+			(xy 66.04 57.15) (xy 66.04 74.93)
+		)
+		(stroke
+			(width 0)
+			(type default)
+		)
+	)
+	(wire
+		(pts
 			(xy 104.14 64.77) (xy 110.49 64.77)
 		)
@@
 	(wire
 		(pts
-			(xy 66.04 45.72) (xy 66.04 74.93)
+			(xy 66.04 45.72) (xy 66.04 57.15)
 		)
 		(stroke
@@
 	(wire
 		(pts
+			(xy 54.61 57.15) (xy 66.04 57.15)
+		)
+		(stroke
+			(width 0)
+			(type default)
+		)
+	)
+	(wire
+		(pts
 			(xy 39.37 66.04) (xy 39.37 77.47)
 		)
@@
 	(wire
 		(pts
+			(xy 74.93 52.07) (xy 74.93 40.64)
+		)
+		(stroke
+			(width 0)
+			(type default)
+		)
+	)
+	(wire
+		(pts
+			(xy 54.61 52.07) (xy 74.93 52.07)
+		)
+		(stroke
+			(width 0)
+			(type default)
+		)
+	)
+	(wire
+		(pts
 			(xy 44.45 104.14) (xy 46.99 104.14)
 		)
@@
 	(wire
 		(pts
-			(xy 74.93 64.77) (xy 74.93 40.64)
+			(xy 74.93 64.77) (xy 74.93 52.07)
 		)
 		(stroke
@@
 			)
 		)
+		(property "Mouser Nr" ""
+			(at 39.37 43.18 0)
+			(effects
+				(font
+					(size 1.27 1.27)
+				)
+				(hide yes)
+			)
+		)
+		(property "Digikey Nr" ""
+			(at 39.37 43.18 0)
+			(effects
+				(font
+					(size 1.27 1.27)
+				)
+				(hide yes)
+			)
+		)
+		(property "FootprintText" ""
+			(at 39.37 43.18 0)
+			(effects
+				(font
+					(size 1.27 1.27)
+				)
+			)
+		)
+		(property "Manufacturer" ""
+			(at 39.37 43.18 0)
+			(effects
+				(font
+					(size 1.27 1.27)
+				)
+				(hide yes)
+			)
+		)
+		(property "ManufacturerNr" ""
+			(at 39.37 43.18 0)
+			(effects
+				(font
+					(size 1.27 1.27)
+				)
+				(hide yes)
+			)
+		)
+		(property "Supplier 1" ""
+			(at 39.37 43.18 0)
+			(effects
+				(font
+					(size 1.27 1.27)
+				)
+				(hide yes)
+			)
+		)
+		(property "Supplier 1 Number" ""
+			(at 39.37 43.18 0)
+			(effects
+				(font
+					(size 1.27 1.27)
+				)
+				(hide yes)
+			)
+		)
+		(property "Supplier 2" ""
+			(at 39.37 43.18 0)
+			(effects
+				(font
+					(size 1.27 1.27)
+				)
+				(hide yes)
+			)
+		)
+		(property "Supplier 2 Number" ""
+			(at 39.37 43.18 0)
+			(effects
+				(font
+					(size 1.27 1.27)
+				)
+				(hide yes)
+			)
+		)
+		(property "Visible 1" ""
+			(at 39.37 43.18 0)
+			(effects
+				(font
+					(size 1.27 1.27)
+				)
+			)
+		)
+		(property "Visible 2" ""
+			(at 39.37 43.18 0)
+			(effects
+				(font
+					(size 1.27 1.27)
+				)
+			)
+		)
 		(pin "S1"
 		)
@@
 		(pin "A7"
 		)
+		(pin "B6"
+		)
+		(pin "B7"
+		)
 		(instances
